File: circuit/battery.kicad_pcb (KiCad board)
At the start: 2 copper layers, 86 x 69 mm, 48 parts, among them J1 Conn_01x02, J2 Conn_01x02, J4 DB15_Male, Q1 PN2222A, SW1 ANT11SF1CQE, U1 TL431LP, U2 AD623AN

Commit message: Started writing documentation
Changed lines of the file:
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@@
     (descr "wire loop with bead as test point, loop diameter2.6mm, hole diameter 1.6mm")
     (tags "test point wire loop bead")
-    (fp_text reference TP1 (at 0.244999 3.175) (layer F.SilkS)
+    (fp_text reference TP1 (at -3.438001 0.127) (layer F.SilkS)
       (effects (font (size 1 1) (thickness 0.15)))
     )
@@
     (descr "wire loop with bead as test point, loop diameter2.6mm, hole diameter 1.6mm")
     (tags "test point wire loop bead")
-    (fp_text reference TP2 (at 0 3.175) (layer F.SilkS)
+    (fp_text reference TP2 (at -3.556 0.127) (layer F.SilkS)
       (effects (font (size 1 1) (thickness 0.15)))
     )
@@
     (descr "wire loop with bead as test point, loop diameter2.6mm, hole diameter 1.6mm")
     (tags "test point wire loop bead")
-    (fp_text reference TP3 (at -0.127 3.175) (layer F.SilkS)
+    (fp_text reference TP3 (at -3.683 0.127) (layer F.SilkS)
       (effects (font (size 1 1) (thickness 0.15)))
     )
@@
   (segment (start 172.055 76.62) (end 177.77 82.335) (width 0.381) (layer B.Cu) (net 17))
   (segment (start 166.975 76.62) (end 172.055 76.62) (width 0.381) (layer B.Cu) (net 17))
-  (segment (start 140.305 63.285) (end 137.765 63.285) (width 0.635) (layer B.Cu) (net 35))
-  (segment (start 142.845 63.285) (end 143.48 62.65) (width 0.635) (layer B.Cu) (net 35))
   (segment (start 137.765 102.02) (end 139.67 102.02) (width 0.381) (layer B.Cu) (net 22))
   (segment (start 136.495 100.75) (end 137.765 102.02) (width 0.381) (layer B.Cu) (net 22))
@@
   (segment (start 137.765 88.05) (end 139.67 86.145) (width 0.381) (layer B.Cu) (net 34))
   (segment (start 135.225 88.05) (end 137.765 88.05) (width 0.381) (layer B.Cu) (net 34))
+  (segment (start 140.305 63.285) (end 137.765 63.285) (width 0.635) (layer B.Cu) (net 35))
+  (segment (start 142.845 63.285) (end 143.48 62.65) (width 0.635) (layer B.Cu) (net 35))
   (segment (start 145.56 75.35) (end 144.115 75.35) (width 0.635) (layer B.Cu) (net 35))
   (segment (start 142.21 73.445) (end 142.21 65.19) (width 0.635) (layer B.Cu) (net 35))
