File: circuit/battery.sch (KiCad schematic (older format))
At the start: 41 parts, among them J1 Conn_01x02, J2 Conn_01x02, J4 DB15_Male, Q1 BS107, SW1 ANT11SF1CQE, U1 TL431LP, U2 AD623AN

Commit message: Final board design; production complete
Parts:
- removed Q1: BS107, Package_TO_SOT_THT:TO-92_Inline_Wide, symbol Transistor_FET:BS107
- added Q1: PN2222A, Package_TO_SOT_THT:TO-92_Inline_Wide, symbol Transistor_BJT:PN2222A
- added R11: 270, Resistor_THT:R_Axial_DIN0207_L6.3mm_D2.5mm_P10.16mm_Horizontal, symbol Device:R
- R8: value 300 -> 270
Connections:
- net ALARM: now also R11.1
- net GND: now also Q1.1 (E)
- net at R8.2, SW1.1 (A): now also Q1.3 (C)
- new net: Q1.2 (B), R11.2
Changed lines of the file:
@@
 U 1 1 61B4ABCC
 P 3950 4750
-F 0 "BZ1" H 3955 5040 50  0000 C CNN
-F 1 "CMI-1295IC-0585T" H 3955 4949 50  0000 C CNN
+F 0 "BZ1" H 4250 4850 50  0000 C CNN
+F 1 "CMI-1295IC-0585T" H 4500 4750 50  0000 C CNN
 F 2 "Buzzer_Beeper:Buzzer_12x9.5RM7.6" V 3925 4850 50  0001 C CNN
 F 3 "~" V 3925 4850 50  0001 C CNN
@@
 P 4550 5350
 F 0 "R8" V 4450 5400 50  0000 C CNN
-F 1 "300" V 4650 5350 50  0000 C CNN
+F 1 "270" V 4650 5350 50  0000 C CNN
 F 2 "Resistor_THT:R_Axial_DIN0207_L6.3mm_D2.5mm_P10.16mm_Horizontal" V 4480 5350 50  0001 C CNN
 F 3 "~" H 4550 5350 50  0001 C CNN
@@
 	4650 2100 4850 2100
 Connection ~ 4850 2100
-$Comp
-L Transistor_FET:BS107 Q1
-U 1 1 61BEC9A9
-P 4350 6000
-F 0 "Q1" H 4555 6046 50  0000 L CNN
-F 1 "BS107" H 4555 5955 50  0000 L CNN
-F 2 "Package_TO_SOT_THT:TO-92_Inline_Wide" H 4550 5925 50  0001 L CIN
-F 3 "http://www.onsemi.com/pub_link/Collateral/BS107-D.PDF" H 4350 6000 50  0001 L CNN
-	1    4350 6000
-	-1   0    0    -1
-$EndComp
 Text GLabel 6000 4300 1    50   Input ~ 0
 IND1
@@
 Wire Wire Line
 	6000 4300 6000 4850
-Wire Wire Line
-	4550 6000 5300 6000
 Text Notes 5150 5750 0    50   ~ 0
 EIO PINS HAVE A 180 OHM SERIES RESISTOR
@@
 U 1 1 61CA8360
 P 4150 5250
-F 0 "SW1" V 4050 4950 50  0000 L CNN
-F 1 "ANT11SF1CQE" V 4200 4700 50  0000 L CNN
+F 0 "SW1" V 4100 4800 50  0000 L CNN
+F 1 "ANT11SF1CQE" V 4200 4550 50  0000 L CNN
 F 2 "_batmon:SW_CIT_ANT_SPDT" H 4150 5250 50  0001 C CNN
 F 3 "~" H 4150 5250 50  0001 C CNN
@@
 Wire Wire Line
 	4100 2200 5550 2200
+$Comp
+L Device:R R11
+U 1 1 61AFC828
+P 4900 6000
+F 0 "R11" V 4800 6050 50  0000 C CNN
+F 1 "270" V 5000 6000 50  0000 C CNN
+F 2 "Resistor_THT:R_Axial_DIN0207_L6.3mm_D2.5mm_P10.16mm_Horizontal" V 4830 6000 50  0001 C CNN
+F 3 "~" H 4900 6000 50  0001 C CNN
+	1    4900 6000
+	0    1    -1   0
+$EndComp
+Wire Wire Line
+	4550 6000 4750 6000
+Wire Wire Line
+	5050 6000 5300 6000
+$Comp
+L Transistor_BJT:PN2222A Q1
+U 1 1 61B090F2
+P 4350 6000
+F 0 "Q1" H 4541 6046 50  0000 L CNN
+F 1 "PN2222A" H 4541 5955 50  0000 L CNN
+F 2 "Package_TO_SOT_THT:TO-92_Inline_Wide" H 4550 5925 50  0001 L CIN
+F 3 "http://www.fairchildsemi.com/ds/PN/PN2222A.pdf" H 4350 6000 50  0001 L CNN
+	1    4350 6000
+	-1   0    0    -1
+$EndComp
 $EndSCHEMATC

Commit message: Placed digikey order
Parts:
- R1: value 500 -> 470
Changed lines of the file:
@@
 P 1200 1300
 F 0 "R1" V 1400 1300 50  0000 C CNN
-F 1 "500" V 1300 1350 50  0000 C CNN
+F 1 "470" V 1300 1350 50  0000 C CNN
 F 2 "Resistor_THT:R_Axial_DIN0207_L6.3mm_D2.5mm_P10.16mm_Horizontal" V 1130 1300 50  0001 C CNN
 F 3 "~" H 1200 1300 50  0001 C CNN

Commit message: Started writing documentation
Other:
- note added: "R4 PROVIDES PROTECTION AGAINST MISWIRING BAT\nC2 RAPIDLY CHARGES THE ADC MUX\nD1 AND D2 PROTECT AGAINST REVERSE POLARITY AND OVER-VOLTAGE\n 100V OVER VOLTAGE DUMPS ABOUT 10mA TO 2.5V"
- note removed: "R4 PROVIDES PROTECTION AGAINST MISWIRING BS\nC2 RAPIDLY CHARGES THE ADC MUX\nD1 AND D2 PROTECT AGAINST REVERSE POLARITY AND OVER-VOLTAGE\n 100V OVER VOLTAGE DUMPS ABOUT 10mA TO 2.5V"
Changed lines of the file:
@@
 U 1 1 619F0792
 P 6450 2850
-F 0 "R15" V 6350 2950 50  0000 C CNN
-F 1 "10K_1%" V 6350 2700 50  0000 C CNN
+F 0 "R15" V 6350 2850 50  0000 C CNN
+F 1 "10K_1%" V 6550 2850 50  0000 C CNN
 F 2 "Resistor_THT:R_Axial_DIN0207_L6.3mm_D2.5mm_P10.16mm_Horizontal" V 6380 2850 50  0001 C CNN
 F 3 "~" H 6450 2850 50  0001 C CNN
@@
 U 1 1 61A830A1
 P 6650 2000
-F 0 "R16" V 6450 2050 50  0000 C CNN
-F 1 "100" V 6550 2050 50  0000 C CNN
+F 0 "R16" V 6550 2000 50  0000 C CNN
+F 1 "100" V 6750 2000 50  0000 C CNN
 F 2 "Resistor_THT:R_Axial_DIN0207_L6.3mm_D2.5mm_P10.16mm_Horizontal" V 6580 2000 50  0001 C CNN
 F 3 "~" H 6650 2000 50  0001 C CNN
@@
 BY ADJUSTING TRIM POT RV1,\nTHE MAXIMUM FULL-SCALE \nVALUE FOR BS (2.44V) MAY BE\nSET TO CORRESPOND TO:\n  MAX:  24.8V\n  NOM: 18.0V\n  MIN: 13.5V
 Text Notes 1250 6700 0    50   ~ 0
-R4 PROVIDES PROTECTION AGAINST MISWIRING BS\nC2 RAPIDLY CHARGES THE ADC MUX\nD1 AND D2 PROTECT AGAINST REVERSE POLARITY AND OVER-VOLTAGE\n  100V OVER VOLTAGE DUMPS ABOUT 10mA TO 2.5V
+R4 PROVIDES PROTECTION AGAINST MISWIRING BAT\nC2 RAPIDLY CHARGES THE ADC MUX\nD1 AND D2 PROTECT AGAINST REVERSE POLARITY AND OVER-VOLTAGE\n  100V OVER VOLTAGE DUMPS ABOUT 10mA TO 2.5V
 Text Notes 3800 3500 0    50   ~ 0
 PARALLEL VOLTAGE DIVIDERS PULL THE SHUNT SIGNAL\nTO THE MIDDLE OF THE UNIPOLAR MEASUREMENT RANGE.  \nTRIM POT RV2 ALLOWS FINE NULL ADJUSTMENT.\nTHE REFERENCE VOLTAGE IS SET TO 1.25V.\nINPUT +/-0.10V SHOULD MAP TO 0.25V TO 2.25V.
@@
 P 4500 2400
 F 0 "D11" V 4450 2500 50  0000 L CNN
-F 1 "1N3595" V 4550 2000 50  0000 L CNN
+F 1 "1N3595" V 4600 2050 50  0000 L CNN
 F 2 "Diode_THT:D_DO-35_SOD27_P7.62mm_Horizontal" H 4500 2400 50  0001 C CNN
 F 3 "~" H 4500 2400 50  0001 C CNN

Commit message: started adding documentation to bmcmd
Parts:
- added C3: 1u, Capacitor_THT:C_Disc_D3.0mm_W1.6mm_P2.50mm, symbol Device:C
Connections:
- net at D11.1 (K), D8.2 (A), RV2.2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: now also C3.1
- net at D3.2 (A), D4.1 (K), R6.1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: now also C3.2
Other:
- note added: "PARALLEL VOLTAGE DIVIDERS PULL THE SHUNT SIGNAL\nTO THE MIDDLE OF THE UNIPOLAR MEASUREMENT RANGE. \nTRIM POT RV2 ALLOWS FINE NULL ADJUSTMENT.\nTHE REFERENCE VOLTAGE IS SET TO 1.25V.\nINPUT +/-0.10V SHOULD MAP TO 0.25V TO 2.25V.\n--> C3 WAS ADDED AFTER BOARD DESIGN"
- note removed: "PARALLEL VOLTAGE DIVIDERS PULL THE SHUNT SIGNAL\nTO THE MIDDLE OF THE UNIPOLAR MEASUREMENT RANGE. \nTRIM POT RV2 ALLOWS FINE NULL ADJUSTMENT.\nTHE REFERENCE VOLTAGE IS SET TO 1.25V.\nINPUT +/-0.10V SHOULD MAP TO 0.25V TO 2.25V."
Changed lines of the file:
@@
 Text Notes 1250 6700 0    50   ~ 0
 R4 PROVIDES PROTECTION AGAINST MISWIRING BAT\nC2 RAPIDLY CHARGES THE ADC MUX\nD1 AND D2 PROTECT AGAINST REVERSE POLARITY AND OVER-VOLTAGE\n  100V OVER VOLTAGE DUMPS ABOUT 10mA TO 2.5V
-Text Notes 3800 3500 0    50   ~ 0
-PARALLEL VOLTAGE DIVIDERS PULL THE SHUNT SIGNAL\nTO THE MIDDLE OF THE UNIPOLAR MEASUREMENT RANGE.  \nTRIM POT RV2 ALLOWS FINE NULL ADJUSTMENT.\nTHE REFERENCE VOLTAGE IS SET TO 1.25V.\nINPUT +/-0.10V SHOULD MAP TO 0.25V TO 2.25V.
+Text Notes 3800 3600 0    50   ~ 0
+PARALLEL VOLTAGE DIVIDERS PULL THE SHUNT SIGNAL\nTO THE MIDDLE OF THE UNIPOLAR MEASUREMENT RANGE.  \nTRIM POT RV2 ALLOWS FINE NULL ADJUSTMENT.\nTHE REFERENCE VOLTAGE IS SET TO 1.25V.\nINPUT +/-0.10V SHOULD MAP TO 0.25V TO 2.25V.\n--> C3 WAS ADDED AFTER BOARD DESIGN
 Wire Wire Line
 	6050 2850 6300 2850
@@
 	2950 3100 3700 3100
 Wire Wire Line
-	3850 1800 4500 1800
+	3850 1800 4300 1800
 Wire Wire Line
 	4100 1350 4100 2200
@@
 	4100 2250 4100 2200
 Wire Wire Line
-	4100 2200 5550 2200
+	4100 2200 4300 2200
 $Comp
 L Device:R R11
@@
 	-1   0    0    -1
 $EndComp
+$Comp
+L Device:C C3
+U 1 1 61C3D466
+P 4300 1950
+F 0 "C3" V 4400 1800 50  0000 C CNN
+F 1 "1u" V 4300 2200 50  0000 C CNN
+F 2 "Capacitor_THT:C_Disc_D3.0mm_W1.6mm_P2.50mm" H 4338 1800 50  0001 C CNN
+F 3 "~" H 4300 1950 50  0001 C CNN
+	1    4300 1950
+	1    0    0    -1
+$EndComp
+Connection ~ 4300 1800
+Wire Wire Line
+	4300 1800 4500 1800
+Wire Wire Line
+	4300 2100 4300 2200
+Connection ~ 4300 2200
+Wire Wire Line
+	4300 2200 5550 2200
 $EndSCHEMATC
